File: pcb/v0/pmod_microsd.kicad_pcb (KiCad board)
At the start: 4 copper layers, 25 x 20.3 mm, 22 parts, among them J4 MICROSD, U1 LSF0108PWR, U2 SN74CB3T3245PWR, U3 SN74LVC1G125DBVR, U7 TLV74018PDBVR

Commit message: add hardware reset
Parts:
- removed R3: 100R, Resistor_SMD:R_0402_1005Metric
- added Q1: SI2301-ZE P-CH, Package_TO_SOT_SMD:SOT-23, B.Cu at (122.3, 102.9)
- added R7: 536R, Resistor_SMD:R_0402_1005Metric, B.Cu at (114.5, 115.8)
- R2: value 20K -> 100K
- moved R2 14.5 mm to (120.0, 103.9), turned to 90 degrees
- moved C3 0.10 mm to (121.0, 105.7)
Connections:
- C26 pad 1: /PWR3V3 -> /PWRSD
- C27 pad 1: /PWR3V3 -> /PWRSD
- J4 pad 4: /PWR3V3 -> /PWRSD
- R2 pad 1: /SDC_CD -> /PWR3V3
- R2 pad 2: /PWR3V3 -> /SD_CD
Routing:
- net /SD_CD: track 10.3 -> 39.9 mm, vias 1 -> 0
- net /PWRSD: track 0.00 -> 23.4 mm, vias 0 -> 2
- net /SD_VSEL: track 25.8 -> 30.2 mm
- net GND: track 28.9 -> 31.1 mm, vias 12 -> 13
- net /PWR3V3: track 22.0 -> 20.1 mm, vias 6 -> 7
- net /SDC_CD: track 5.44 -> 6.53 mm
- net /PWR1V8: track 10.5 -> 11.1 mm
- added copper zone on B.Cu, net GND
- added copper zone on F.Cu, net GND

Commit message: update values
Parts:
- R2: value 100K -> 20K
- R7: value 536R -> 1K
Changed lines of the file:
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@@
 			(at -3.5 0 90)
 			(layer "Dwgs.User")
-			(hide yes)
 			(effects
 				(font
-					(size 1.016 1.016)
+					(size 0.5 0.5)
 					(thickness 0.2032)
 				)
@@
 			(at 4.3 -10.4 90)
 			(layer "Dwgs.User")
-			(hide yes)
 			(effects
 				(font
-					(size 0.3 0.3)
+					(size 0.5 0.5)
 					(thickness 0.03)
 				)
@@
 		)
 		(property "Value" "DNP"
-			(at 0 -2.1 0)
+			(at -2.55 -0.25 0)
 			(layer "B.Fab")
-			(hide yes)
 			(effects
 				(font
-					(size 1 1)
+					(size 0.5 0.5)
 					(thickness 0.15)
 				)
@@
 		)
 		(property "Value" "1K"
-			(at 0 -2.1 0)
+			(at -1.1 0 0)
 			(layer "B.Fab")
-			(hide yes)
 			(effects
 				(font
-					(size 1 1)
+					(size 0.5 0.5)
 					(thickness 0.15)
 				)
@@
 		)
 		(property "Value" "1uF"
-			(at 0 -1.16 90)
+			(at -0.02 0.8 90)
 			(layer "B.Fab")
-			(hide yes)
 			(effects
 				(font
-					(size 1 1)
+					(size 0.5 0.5)
 					(thickness 0.15)
 				)
@@
 			)
 		)
-		(property "Value" "100K"
-			(at 0 -1.17 90)
+		(property "Value" "20K"
+			(at 1.8 0 90)
 			(layer "B.Fab")
-			(hide yes)
 			(effects
 				(font
-					(size 1 1)
+					(size 0.5 0.5)
 					(thickness 0.15)
 				)
@@
 		)
 		(property "Value" "10uF"
-			(at 0 -1.16 90)
+			(at -0.05 1.3 0)
 			(layer "B.Fab")
-			(hide yes)
 			(effects
 				(font
-					(size 1 1)
+					(size 0.5 0.5)
 					(thickness 0.15)
 				)
@@
 			)
 		)
-		(property "Value" "536R"
-			(at 0 -1.17 0)
+		(property "Value" "1K"
+			(at -0.05 -0.7 0)
 			(layer "B.Fab")
-			(hide yes)
 			(effects
 				(font
-					(size 1 1)
+					(size 0.5 0.5)
 					(thickness 0.15)
 				)
@@
 		)
 		(property "Value" "200K"
-			(at 0 -1.17 0)
+			(at 1.75 0.05 0)
 			(layer "B.Fab")
-			(hide yes)
 			(effects
 				(font
-					(size 1 1)
+					(size 0.5 0.5)
 					(thickness 0.15)
 				)
@@
 		)
 		(property "Value" "SN74CB3T3245PWR"
-			(at 0 -4.2 0)
+			(at -0.15 -3.95 180)
 			(layer "B.Fab")
-			(hide yes)
 			(effects
 				(font
-					(size 1 1)
+					(size 0.5 0.5)
 					(thickness 0.15)
 				)
@@
 			(at 0.75 0 0)
 			(layer "B.SilkS")
-			(hide yes)
 			(effects
 				(font
-					(size 1.524 1.524)
+					(size 0.5 0.5)
 					(thickness 0.3)
 				)
@@
 		)
 		(property "Value" "100nF"
-			(at 0 -1.16 90)
+			(at -0.08 -1.5 0)
 			(layer "B.Fab")
-			(hide yes)
 			(effects
 				(font
-					(size 1 1)
+					(size 0.5 0.5)
 					(thickness 0.15)
 				)
@@
 		)
 		(property "Value" "100nF"
-			(at 0 -1.16 90)
+			(at -1.86 0 90)
 			(layer "B.Fab")
-			(hide yes)
 			(effects
 				(font
-					(size 1 1)
+					(size 0.5 0.5)
 					(thickness 0.15)
 				)
@@
 		)
 		(property "Value" "SN74LVC1G125DBVR"
-			(at 0 -2.4 0)
+			(at -2.75 2.34 0)
 			(layer "B.Fab")
-			(hide yes)
 			(effects
 				(font
-					(size 1 1)
+					(size 0.5 0.5)
 					(thickness 0.15)
 				)
@@
 		)
 		(property "Value" "LSF0108PWR"
-			(at 0 -4.2 0)
+			(at -1.65 -0.35 -90)
 			(layer "B.Fab")
-			(hide yes)
 			(effects
 				(font
-					(size 1 1)
+					(size 0.5 0.5)
 					(thickness 0.15)
 				)
@@
 		)
 		(property "Value" "100nF"
-			(at 0 -1.16 0)
+			(at 1.9 0 0)
 			(layer "B.Fab")
-			(hide yes)
 			(effects
 				(font
-					(size 1 1)
+					(size 0.5 0.5)
 					(thickness 0.15)
 				)
@@
 		)
 		(property "Value" "1K"
-			(at 0 -2.1 0)
+			(at 1.2 0.05 0)
 			(layer "B.Fab")
-			(hide yes)
 			(effects
 				(font
-					(size 1 1)
+					(size 0.5 0.5)
 					(thickness 0.15)
 				)
@@
 		)
 		(property "Value" "1uF"
-			(at 0 -1.16 90)
+			(at -1.37 0 90)
 			(layer "B.Fab")
-			(hide yes)
 			(effects
 				(font
-					(size 1 1)
+					(size 0.5 0.5)
 					(thickness 0.15)
 				)
@@
 		)
 		(property "Value" "100nF"
-			(at 0 -1.16 0)
+			(at 1.875 0.025 0)
 			(layer "B.Fab")
-			(hide yes)
 			(effects
 				(font
-					(size 1 1)
+					(size 0.5 0.5)
 					(thickness 0.15)
 				)
@@
 		)
 		(property "Value" "DNP"
-			(at 0 -2.1 0)
+			(at -2.6 -0.3 0)
 			(layer "B.Fab")
-			(hide yes)
 			(effects
 				(font
-					(size 1 1)
+					(size 0.5 0.5)
 					(thickness 0.15)
 				)
@@
 		)
 		(property "Value" "10K"
-			(at 0 -1.17 90)
+			(at -0.05 0.7 90)
 			(layer "B.Fab")
-			(hide yes)
 			(effects
 				(font
-					(size 1 1)
+					(size 0.5 0.5)
 					(thickness 0.15)
 				)
@@
 		)
 		(property "Value" "SI2301-ZE P-CH"
-			(at 0 -2.4 90)
+			(at -2.15 -2.1625 90)
 			(layer "B.Fab")
-			(hide yes)
 			(effects
 				(font
-					(size 1 1)
+					(size 0.5 0.5)
 					(thickness 0.15)
 				)
@@
 		)
 		(property "Value" "TLV74018PDBVR"
-			(at 0 -2.4 0)
+			(at 1.7625 2.24 0)
 			(layer "B.Fab")
-			(hide yes)
 			(effects
 				(font
-					(size 1 1)
+					(size 0.5 0.5)
 					(thickness 0.15)
 				)

Commit message: update readme & schematics
Parts:
- RN2, RN4: value 1K -> 510R
Changed lines of the file:
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@@
 			)
 		)
-		(property "Value" "1K"
+		(property "Value" "510R"
 			(at -1.1 0 0)
 			(layer "B.Fab")
@@
 			)
 		)
-		(property "Value" "1K"
+		(property "Value" "510R"
 			(at 1.2 0.05 0)
 			(layer "B.Fab")
