File: pcb/v0/pmod_microsd.kicad_sch (KiCad schematic)
At the start: 21 parts, among them J4 MICROSD, U1 LSF0108PWR, U2 SN74CB3T3245PWR, U3 SN74LVC1G125DBVR, U7 TLV74018PDBVR

Commit message: add hardware reset
Parts:
- added Q1: SI2301-ZE P-CH, Package_TO_SOT_SMD:SOT-23, symbol Transistor_FET:BSS84
- added R7: 1K, Resistor_SMD:R_0402_1005Metric, symbol Device:R
- R3: value 100R -> 270R
Connections:
- net PWR3V3: now also R2.1, Q1.2 (S); no longer C26.1, C27.1, J4.4 (VDD), R2.2
- net SDC_CD: now also R7.1; no longer R2.1, R3.1
- new net: Q1.1 (G), R2.2, R3.1, R7.2
- new net PWRSD: C26.1, C27.1, J4.4 (VDD), Q1.3 (D)
Other:
- note added: "SD_CD is pulled high when no card is inserted. SD_CD is pulled low when a card is inserted. PWRSD shuts off when SD_CD is driven to 3.3V."
- moved on the sheet: C35, C39, R4, U7

Commit message: update values
Parts:
- removed R3: 270R, Resistor_SMD:R_0402_1005Metric, symbol Device:R
- R7: value 1K -> 536
- RN2, RN4: value 1K -> 510R
Connections:
- net SD_CD: now also Q1.1 (G), R2.2, R7.2
Changed lines of the file:
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@@
 	)
 	(junction
-		(at 157.48 87.63)
+		(at 132.08 171.45)
 		(diameter 0)
 		(color 0 0 0 0)
 	)
 	(junction
-		(at 132.08 171.45)
+		(at 157.48 87.63)
 		(diameter 0)
 		(color 0 0 0 0)
@@
 	(wire
 		(pts
-			(xy 132.08 171.45) (xy 140.97 171.45)
+			(xy 129.54 171.45) (xy 132.08 171.45)
 		)
 		(stroke
@@
 	(wire
 		(pts
+			(xy 132.08 171.45) (xy 140.97 171.45)
+		)
+		(stroke
+			(width 0)
+			(type default)
+		)
+	)
+	(wire
+		(pts
 			(xy 44.45 111.76) (xy 87.63 111.76)
 		)
@@
 	(wire
 		(pts
+			(xy 132.08 149.86) (xy 132.08 171.45)
+		)
+		(stroke
+			(width 0)
+			(type default)
+		)
+	)
+	(wire
+		(pts
 			(xy 36.83 168.91) (xy 54.61 168.91)
 		)
@@
 	(wire
 		(pts
-			(xy 132.08 166.37) (xy 132.08 171.45)
-		)
-		(stroke
-			(width 0)
-			(type default)
-		)
-	)
-	(wire
-		(pts
 			(xy 63.5 49.53) (xy 81.28 49.53)
 		)
@@
 	(wire
 		(pts
-			(xy 132.08 149.86) (xy 132.08 158.75)
-		)
-		(stroke
-			(width 0)
-			(type default)
-		)
-	)
-	(wire
-		(pts
 			(xy 223.52 129.54) (xy 223.52 127)
 		)
@@
 		)
 	)
-	(wire
-		(pts
-			(xy 129.54 171.45) (xy 132.08 171.45)
-		)
-		(stroke
-			(width 0)
-			(type default)
-		)
-	)
 	(text "SD_CD is pulled high when no card is inserted.\n\nSD_CD is pulled low when a card is inserted.\n\nPWRSD shuts off when SD_CD is driven to 3.3V."
 		(exclude_from_sim no)
@@
 			)
 		)
-		(property "Value" "1K"
+		(property "Value" "536"
 			(at 124.4601 173.99 0)
 			(effects
@@
 	)
 	(symbol
-		(lib_id "Device:R")
-		(at 132.08 162.56 180)
-		(unit 1)
-		(exclude_from_sim no)
-		(in_bom yes)
-		(on_board yes)
-		(dnp no)
-		(property "Reference" "R3"
-			(at 124.46 161.29 0)
-			(effects
-				(font
-					(size 1.27 1.27)
-				)
-				(justify right)
-			)
-		)
-		(property "Value" "270R"
-			(at 124.46 163.83 0)
-			(effects
-				(font
-					(size 1.27 1.27)
-				)
-				(justify right)
-			)
-		)
-		(property "Footprint" "Resistor_SMD:R_0402_1005Metric"
-			(at 133.858 162.56 90)
-			(effects
-				(font
-					(size 1.27 1.27)
-				)
-				(hide yes)
-			)
-		)
-		(property "Datasheet" "~"
-			(at 132.08 162.56 0)
-			(effects
-				(font
-					(size 1.27 1.27)
-				)
-				(hide yes)
-			)
-		)
-		(property "Description" "Resistor"
-			(at 132.08 162.56 0)
-			(effects
-				(font
-					(size 1.27 1.27)
-				)
-				(hide yes)
-			)
-		)
-		(pin "1"
-		)
-		(pin "2"
-		)
-		(instances
-			(project "pmod_microsd"
-				(path "/f68096f2-5bd7-4426-aed8-a7a28447e5be"
-					(reference "R3")
-					(unit 1)
-				)
-			)
-		)
-	)
-	(symbol
 		(lib_id "Device:R_Pack04")
 		(at 140.97 92.71 0)
@@
 			)
 		)
-		(property "Value" "1K"
+		(property "Value" "510R"
 			(at 55.88 91.4401 0)
 			(effects
@@
 			)
 		)
-		(property "Value" "1K"
+		(property "Value" "510R"
 			(at 154.94 93.9799 0)
 			(effects

Commit message: update readme & schematics
Parts:
- R7: value 536 -> 1K
Changed lines of the file:
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@@
 			)
 		)
-		(property "Value" "536"
+		(property "Value" "1K"
 			(at 124.4601 173.99 0)
 			(effects
